Commit message: Redesign ball chaser robot

File: project02/src/my_robot/urdf/my_robot.xacro (robot description, xacro)
@@ -8,9 +8,9 @@
     <child link="chassis" />
   </joint>
-  <link name='chassis'>
-    <pose>0 0 0.1 0 0 0</pose>
+  <link name="chassis">
+    <pose>0 0 0.1 0 0 0 </pose>
     <inertial>
+      <origin xyz="0.0 0.0 0.0" rpy="0.0 0.0 0.0"/>
       <mass value="15.0"/>
-      <origin xyz="0.0 0 0" rpy=" 0 0 0"/>
       <inertia
           ixx="0.1" ixy="0" ixz="0"
@@ -19,16 +19,16 @@
       />
     </inertial>
-    <collision name='collision'>
-      <origin xyz="0 0 0" rpy=" 0 0 0"/>
+    <visual name='chassis_visual'>
+      <origin xyz="0.0 0.0 0.0" rpy="0.0 0.0 0.0"/>
       <geometry>
-        <box size=".4 .2 .1"/>
+        <cylinder radius="0.2" length="0.1"/>
+      </geometry>
+    </visual>
+    <collision name='chassis_collision'>
+      <origin xyz="0.0 0.0 0.0" rpy="0.0 0.0 0.0"/>
+      <geometry>
+        <cylinder radius="0.2" length="0.1"/>
       </geometry>
     </collision>
-    <visual name='chassis_visual'>
-      <origin xyz="0 0 0" rpy=" 0 0 0"/>
-      <geometry>
-        <box size=".4 .2 .1"/>
-      </geometry>
-    </visual>
     <collision name='back_caster_collision'>
       <origin xyz="-0.15 0 -0.05" rpy=" 0 0 0"/>
@@ -60,5 +60,5 @@
       <origin xyz="0.0 0 0" rpy="  0 1.5707 1.5707"/>
       <geometry>
-        <cylinder radius="0.1" length="0.05"/>
+        <cylinder radius="0.075" length="0.05"/>
       </geometry>
     </collision>
@@ -67,7 +67,7 @@
       <origin xyz="0.0 0 0" rpy="  0 1.5707 1.5707"/>
       <inertia
-          ixx="0.1" ixy="0" ixz="0"
-          iyy="0.1" iyz="0"
-          izz="0.1"
+          ixx="0.075" ixy="0" ixz="0"
+          iyy="0.075" iyz="0"
+          izz="0.075"
       />
     </inertial>
@@ -75,10 +75,10 @@
       <origin xyz="0.0 0 0" rpy="  0 1.5707 1.5707"/>
       <geometry>
-        <cylinder radius="0.1" length="0.05"/>
+        <cylinder radius="0.075" length="0.05"/>
       </geometry>
     </visual>
   </link>
   <joint type="continuous" name="left_wheel_hinge">
-    <origin xyz="0 0.15 0" rpy="0 0 0"/>
+    <origin xyz="0 0.23 -0.025" rpy="0 0 0"/>
     <child link="left_wheel"/>
     <parent link="chassis"/>
@@ -91,5 +91,5 @@
       <origin xyz="0.0 0 0" rpy="  0 1.5707 1.5707"/>
       <geometry>
-        <cylinder radius="0.1" length="0.05"/>
+        <cylinder radius="0.075" length="0.05"/>
       </geometry>
     </collision>
@@ -98,7 +98,7 @@
       <origin xyz="0.0 0 0" rpy="  0 1.5707 1.5707"/>
       <inertia
-          ixx="0.1" ixy="0" ixz="0"
-          iyy="0.1" iyz="0"
-          izz="0.1"
+          ixx="0.075" ixy="0" ixz="0"
+          iyy="0.075" iyz="0"
+          izz="0.075"
       />
     </inertial>
@@ -106,10 +106,10 @@
       <origin xyz="0.0 0 0" rpy="  0 1.5707 1.5707"/>
       <geometry>
-        <cylinder radius="0.1" length="0.05"/>
+        <cylinder radius="0.075" length="0.05"/>
       </geometry>
     </visual>
   </link>
   <joint type="continuous" name="right_wheel_hinge">
-    <origin xyz="0 -0.15 0" rpy="0 0 0"/>
+    <origin xyz="0 -0.23 -0.025" rpy="0 0 0"/>
     <child link="right_wheel"/>
     <parent link="chassis"/>
@@ -171,5 +171,5 @@
   </link>
   <joint name="hokuyo_joint" type="fixed">
-    <origin xyz="0.15 0 0.1" rpy="0 0 0"/>
+    <origin xyz="0.15 0 0.08" rpy="0 0 0"/>
     <child link="hokuyo"/>
     <parent link="chassis"/>
@@ -177,14 +177,14 @@
   </joint>
   <gazebo reference="left_wheel">
+    <material>Gazebo/Turquoise</material>
+  </gazebo>
+  <gazebo reference="right_wheel">
+    <material>Gazebo/Turquoise</material>
+  </gazebo>
+  <gazebo reference="camera">
     <material>Gazebo/Green</material>
   </gazebo>
-  <gazebo reference="right_wheel">
-    <material>Gazebo/Green</material>
-  </gazebo>
-  <gazebo reference="camera">
-    <material>Gazebo/Red</material>
-  </gazebo>
   <gazebo reference="chassis">
-    <material>Gazebo/Blue</material>
+    <material>Gazebo/Purple</material>
   </gazebo>
 </robot>
